Commit message: Add files via upload

File: hexbot/urdf/test.urdf (robot description, URDF)
Before this commit: robot hexbot, 17 links, 16 joints
Joints:
- joint fingerleft_tohand: limit lower=0.0 upper=0.04 effort=20 velocity=0.2 -> (none); type prismatic -> fixed
- joint fingerright_tohand: limit lower=-0.04 upper=0 effort=20 velocity=0.2 -> (none); type prismatic -> fixed
